Commit message: commit part1

File: src/rob_description/urdf/robot_model.urdf.xacro (robot description, xacro)
@@ -13,5 +13,5 @@
         <parent link="base_link" />
         <child link = "gps_frame" />
-        <origin xyz="0.0 0.0 0.450" rpy="1.570796 0.0 3.141291" />
+        <origin xyz="0.0 0.0 0.450" rpy="0.0 0.0 -1.5708" />
     </joint>
     <link name="gps_frame" />
@@ -20,5 +20,5 @@
         <parent link="base_link" />
         <child link = "lidar_front_frame" />
-        <origin xyz="0.487 -0.255 0.0" rpy="1.570796 0.0 2.357016" />
+        <origin xyz="0.487 -0.255 0.0" rpy="0.0 0.0 -0.7859" />
     </joint>
     <link name="lidar_front_frame" />
@@ -27,5 +27,5 @@
         <parent link="base_link" />
         <child link = "lidar_back_frame" />
-        <origin xyz="-0.487 0.255 0.0" rpy="1.570796 0.0 -0.78523" />
+        <origin xyz="-0.487 0.255 0.0" rpy="0.0 0.0 2.3557" />
     </joint>
     <link name="lidar_back_frame" />
@@ -34,5 +34,5 @@
         <parent link="base_link" />
         <child link = "imu_frame" />
-        <origin xyz="0.0 0.0 0.450" rpy="1.570796 0.0 3.141291" />
+        <origin xyz="0.0 0.0 0.450" rpy="0.0 0.0 -1.5708" />
     </joint>
     <link name="imu_frame" />
